File: hardware/SMD/relayExtension.kicad_pcb (KiCad board)
At the start: 2 copper layers, 57 x 58 mm, 38 parts, among them J1 Screw_Terminal_01x03, J10 Screw_Terminal_01x03, J11 Screw_Terminal_01x03, J12 Screw_Terminal_01x03, J2 Screw_Terminal_01x03, J3 Screw_Terminal_01x03, J4 Screw_Terminal_01x03, J5 Screw_Terminal_01x03, J6 Screw_Terminal_01x03, J7 Screw_Terminal_01x03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

Commit message: added data to readme.md
Connections:
- net Net-(J11-Pin_1) renamed /relay4/NC1
- net Net-(J11-Pin_2) renamed /relay4/COM1
- net Net-(J11-Pin_3) renamed /relay4/NO1
- net Net-(J12-Pin_1) renamed /relay4/NC2
- net Net-(J12-Pin_2) renamed /relay4/COM2
- net Net-(J12-Pin_3) renamed /relay4/NO2
- net Net-(J3-Pin_1) renamed /relay2/NC1
- net Net-(J3-Pin_2) renamed /relay2/COM1
- net Net-(J3-Pin_3) renamed /relay2/NO1
- net Net-(J4-Pin_1) renamed /relay1/NC1
- net Net-(J4-Pin_2) renamed /relay1/COM1
- net Net-(J4-Pin_3) renamed /relay1/NO1
- net Net-(J5-Pin_1) renamed /relay1/NC2
- net Net-(J5-Pin_2) renamed /relay1/COM2
- net Net-(J5-Pin_3) renamed /relay1/NO2
- net Net-(J6-Pin_1) renamed /relay2/NC2
- net Net-(J6-Pin_2) renamed /relay2/COM2
- net Net-(J6-Pin_3) renamed /relay2/NO2
- net Net-(J8-Pin_1) renamed /relay3/NC1
- net Net-(J8-Pin_2) renamed /relay3/COM1
- net Net-(J8-Pin_3) renamed /relay3/NO1
- net Net-(J9-Pin_1) renamed /relay3/NC2
- net Net-(J9-Pin_2) renamed /relay3/COM2
- net Net-(J9-Pin_3) renamed /relay3/NO2
