File: hardware/General-Purpose-THT/relay.kicad_sch (KiCad schematic)
At the start: 9 parts, among them J1 Screw_Terminal_01x03, J4 Screw_Terminal_01x03, J5 Screw_Terminal_01x03, K201 G5V-1, K202 G5V-1

Commit message: redid the through-hole relay pcb
Connections:
- net at J5.1 (Pin_1): now also K202.10; no longer K202.1
- net at J5.3 (Pin_3): now also K202.1; no longer K202.10
Changed lines of the file:
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@@
 	(label "Coil2"
 		(at 113.03 71.12 0)
-		(fields_autoplaced yes)
 		(effects
 			(font
@@
 	(label "Coil2"
 		(at 133.35 53.34 180)
-		(fields_autoplaced yes)
 		(effects
 			(font
@@
 	(label "Coil1"
 		(at 113.03 66.04 0)
-		(fields_autoplaced yes)
 		(effects
 			(font
@@
 	(label "Coil1"
 		(at 135.89 90.17 180)
-		(fields_autoplaced yes)
 		(effects
 			(font
@@
 					(unit 1)
 				)
-				(path "/e7280eb5-1386-47ea-974c-c755a08b04e7/5b58b096-6dbe-4801-824f-a9589771fa81"
-					(reference "JP401")
-					(unit 1)
-				)
-				(path "/e7280eb5-1386-47ea-974c-c755a08b04e7/8ed02587-de5d-4e4c-b198-ec2f04219e8a"
-					(reference "JP501")
-					(unit 1)
-				)
-				(path "/e7280eb5-1386-47ea-974c-c755a08b04e7/991e30e4-9d55-4765-b468-3531f42cf09b"
-					(reference "JP301")
-					(unit 1)
-				)
 			)
 		)
@@
 					(unit 1)
 				)
-				(path "/e7280eb5-1386-47ea-974c-c755a08b04e7/5b58b096-6dbe-4801-824f-a9589771fa81"
-					(reference "#PWR09")
-					(unit 1)
-				)
-				(path "/e7280eb5-1386-47ea-974c-c755a08b04e7/8ed02587-de5d-4e4c-b198-ec2f04219e8a"
-					(reference "#PWR012")
-					(unit 1)
-				)
-				(path "/e7280eb5-1386-47ea-974c-c755a08b04e7/991e30e4-9d55-4765-b468-3531f42cf09b"
-					(reference "#PWR06")
-					(unit 1)
-				)
 			)
 		)
@@
 					(unit 1)
 				)
-				(path "/e7280eb5-1386-47ea-974c-c755a08b04e7/5b58b096-6dbe-4801-824f-a9589771fa81"
-					(reference "#PWR07")
-					(unit 1)
-				)
-				(path "/e7280eb5-1386-47ea-974c-c755a08b04e7/8ed02587-de5d-4e4c-b198-ec2f04219e8a"
-					(reference "#PWR010")
-					(unit 1)
-				)
-				(path "/e7280eb5-1386-47ea-974c-c755a08b04e7/991e30e4-9d55-4765-b468-3531f42cf09b"
-					(reference "#PWR04")
-					(unit 1)
-				)
 			)
 		)
@@
 					(unit 1)
 				)
-				(path "/e7280eb5-1386-47ea-974c-c755a08b04e7/5b58b096-6dbe-4801-824f-a9589771fa81"
-					(reference "#PWR08")
-					(unit 1)
-				)
-				(path "/e7280eb5-1386-47ea-974c-c755a08b04e7/8ed02587-de5d-4e4c-b198-ec2f04219e8a"
-					(reference "#PWR011")
-					(unit 1)
-				)
-				(path "/e7280eb5-1386-47ea-974c-c755a08b04e7/991e30e4-9d55-4765-b468-3531f42cf09b"
-					(reference "#PWR05")
-					(unit 1)
-				)
 			)
 		)
@@
 					(unit 1)
 				)
-				(path "/e7280eb5-1386-47ea-974c-c755a08b04e7/5b58b096-6dbe-4801-824f-a9589771fa81"
-					(reference "J7")
-					(unit 1)
-				)
-				(path "/e7280eb5-1386-47ea-974c-c755a08b04e7/8ed02587-de5d-4e4c-b198-ec2f04219e8a"
-					(reference "J10")
-					(unit 1)
-				)
-				(path "/e7280eb5-1386-47ea-974c-c755a08b04e7/991e30e4-9d55-4765-b468-3531f42cf09b"
-					(reference "J2")
-					(unit 1)
-				)
 			)
 		)
@@
 		(lib_id "Connector:Screw_Terminal_01x03")
 		(at 171.45 100.33 0)
-		(unit 1)
-		(exclude_from_sim no)
-		(in_bom yes)
-		(on_board yes)
-		(dnp no)
-		(fields_autoplaced yes)
+		(mirror x)
+		(unit 1)
+		(exclude_from_sim no)
+		(in_bom yes)
+		(on_board yes)
+		(dnp no)
 		(property "Reference" "J5"
-			(at 173.99 100.3299 0)
+			(at 173.99 100.3301 0)
 			(effects
 				(font
@@
 		)
 		(property "Value" "Screw_Terminal_01x03"
-			(at 171.45 106.68 0)
+			(at 171.45 93.98 0)
 			(effects
 				(font
@@
 				(path "/e7280eb5-1386-47ea-974c-c755a08b04e7/41bba28a-ec8f-4007-b6c6-6cd3fe4f31f4"
 					(reference "J5")
-					(unit 1)
-				)
-				(path "/e7280eb5-1386-47ea-974c-c755a08b04e7/5b58b096-6dbe-4801-824f-a9589771fa81"
-					(reference "J9")
-					(unit 1)
-				)
-				(path "/e7280eb5-1386-47ea-974c-c755a08b04e7/8ed02587-de5d-4e4c-b198-ec2f04219e8a"
-					(reference "J12")
-					(unit 1)
-				)
-				(path "/e7280eb5-1386-47ea-974c-c755a08b04e7/991e30e4-9d55-4765-b468-3531f42cf09b"
-					(reference "J6")
 					(unit 1)
 				)
@@
 					(unit 1)
 				)
-				(path "/e7280eb5-1386-47ea-974c-c755a08b04e7/5b58b096-6dbe-4801-824f-a9589771fa81"
-					(reference "R401")
-					(unit 1)
-				)
-				(path "/e7280eb5-1386-47ea-974c-c755a08b04e7/8ed02587-de5d-4e4c-b198-ec2f04219e8a"
-					(reference "R501")
-					(unit 1)
-				)
-				(path "/e7280eb5-1386-47ea-974c-c755a08b04e7/991e30e4-9d55-4765-b468-3531f42cf09b"
-					(reference "R301")
-					(unit 1)
-				)
 			)
 		)
@@
 					(unit 1)
 				)
-				(path "/e7280eb5-1386-47ea-974c-c755a08b04e7/5b58b096-6dbe-4801-824f-a9589771fa81"
-					(reference "J8")
-					(unit 1)
-				)
-				(path "/e7280eb5-1386-47ea-974c-c755a08b04e7/8ed02587-de5d-4e4c-b198-ec2f04219e8a"
-					(reference "J11")
-					(unit 1)
-				)
-				(path "/e7280eb5-1386-47ea-974c-c755a08b04e7/991e30e4-9d55-4765-b468-3531f42cf09b"
-					(reference "J3")
-					(unit 1)
-				)
 			)
 		)
@@
 					(unit 1)
 				)
-				(path "/e7280eb5-1386-47ea-974c-c755a08b04e7/5b58b096-6dbe-4801-824f-a9589771fa81"
-					(reference "K401")
-					(unit 1)
-				)
-				(path "/e7280eb5-1386-47ea-974c-c755a08b04e7/8ed02587-de5d-4e4c-b198-ec2f04219e8a"
-					(reference "K501")
-					(unit 1)
-				)
-				(path "/e7280eb5-1386-47ea-974c-c755a08b04e7/991e30e4-9d55-4765-b468-3531f42cf09b"
-					(reference "K301")
-					(unit 1)
-				)
 			)
 		)
@@
 					(unit 1)
 				)
-				(path "/e7280eb5-1386-47ea-974c-c755a08b04e7/5b58b096-6dbe-4801-824f-a9589771fa81"
-					(reference "R402")
-					(unit 1)
-				)
-				(path "/e7280eb5-1386-47ea-974c-c755a08b04e7/8ed02587-de5d-4e4c-b198-ec2f04219e8a"
-					(reference "R502")
-					(unit 1)
-				)
-				(path "/e7280eb5-1386-47ea-974c-c755a08b04e7/991e30e4-9d55-4765-b468-3531f42cf09b"
-					(reference "R302")
-					(unit 1)
-				)
 			)
 		)
@@
 					(unit 1)
 				)
-				(path "/e7280eb5-1386-47ea-974c-c755a08b04e7/5b58b096-6dbe-4801-824f-a9589771fa81"
-					(reference "K402")
-					(unit 1)
-				)
-				(path "/e7280eb5-1386-47ea-974c-c755a08b04e7/8ed02587-de5d-4e4c-b198-ec2f04219e8a"
-					(reference "K502")
-					(unit 1)
-				)
-				(path "/e7280eb5-1386-47ea-974c-c755a08b04e7/991e30e4-9d55-4765-b468-3531f42cf09b"
-					(reference "K302")
-					(unit 1)
-				)
 			)
 		)
@@
 					(unit 1)
 				)
-				(path "/e7280eb5-1386-47ea-974c-c755a08b04e7/5b58b096-6dbe-4801-824f-a9589771fa81"
-					(reference "JP402")
-					(unit 1)
-				)
-				(path "/e7280eb5-1386-47ea-974c-c755a08b04e7/8ed02587-de5d-4e4c-b198-ec2f04219e8a"
-					(reference "JP502")
-					(unit 1)
-				)
-				(path "/e7280eb5-1386-47ea-974c-c755a08b04e7/991e30e4-9d55-4765-b468-3531f42cf09b"
-					(reference "JP302")
-					(unit 1)
-				)
