File: hardware/General-Purpose-THT/General-Purpose-THT.kicad_pcb (KiCad board)
At the start: 2 copper layers, 56.5 x 13 mm, 11 parts, among them J1 Screw_Terminal_01x03, J4 Screw_Terminal_01x03, J5 Screw_Terminal_01x03, K201 G5V-1, K202 G5V-1

Commit message: finalized relays repo. Yet to do manual. Release is ready togo
Other:
- board size 56.5 x 13 mm -> 56.5 x 15 mm
Changed lines of the file:
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@@
 	)
 	(footprint "MountingHole:MountingHole_3.2mm_M3"
-		(locked yes)
 		(layer "F.Cu")
 		(at 136.5 64)
@@
 	)
 	(footprint "Symbol:OSHW-Logo2_9.8x8mm_SilkScreen"
-		(locked yes)
 		(layer "B.Cu")
 		(at 130.048 65.151 -90)
@@
 	)
 	(gr_line
-		(start 159.5 70.5)
-		(end 159.5 57.5)
+		(start 159.5 71.5)
+		(end 159.5 56.5)
 		(stroke
 			(width 0.1)
@@
 	)
 	(gr_line
-		(start 103 70.5)
-		(end 159.5 70.5)
+		(start 103 71.5)
+		(end 159.5 71.5)
 		(stroke
 			(width 0.1)
@@
 	)
 	(gr_line
-		(start 103 57.5)
-		(end 159.5 57.5)
+		(start 103 56.5)
+		(end 159.5 56.5)
 		(stroke
 			(width 0.1)
@@
 	)
 	(gr_line
-		(start 103 57.5)
-		(end 103 70.5)
+		(start 103 56.5)
+		(end 103 71.5)
 		(stroke
 			(width 0.1)
@@
 	)
 	(gr_text "likely 1 unit will cost 4,50 to manufactor and this is en masse"
-		(locked yes)
 		(at 119.25 53.70782 0)
 		(layer "Dwgs.User")
@@
 	)
 	(gr_text "55 ct screw terminal, 2x 66ct relay\n1x 35ct male plug left side\nthe plugs are around 50 cents.\n2,70 components"
-		(locked yes)
 		(at 121 50.5 0)
 		(layer "Dwgs.User")
@@
 	(dimension
 		(type aligned)
-		(locked yes)
 		(layer "Dwgs.User")
 		(pts
-			(xy 159.5 70.5) (xy 159.5 57.5)
+			(xy 159.5 71.5) (xy 159.5 56.5)
 		)
 		(height 7)
-		(gr_text "13,0000 mm"
-			(locked yes)
+		(gr_text "15,0000 mm"
 			(at 165.35 64 90)
 			(layer "Dwgs.User")
@@
 		(net 3)
 		(net_name "+12V")
-		(locked yes)
 		(layer "F.Cu")
 		(hatch edge 0.5)
