File: hardware/General-Purpose-SMD/General-Purpose-SMD.kicad_pcb (KiCad board)
At the start: 2 copper layers, 56 x 17 mm, 8 parts, among them J1 Screw_Terminal_01x03, J4 Screw_Terminal_01x03, J5 Screw_Terminal_01x03, K1 G6K-2F-Y-TR DC12, K2 G6K-2F-Y-TR DC12

Commit message: finalized relays repo. Yet to do manual. Release is ready togo
Parts:
- added REF**: OSHW-Logo2_9.8x8mm_SilkScreen, Symbol:OSHW-Logo2_9.8x8mm_SilkScreen, B.Cu at (120.4, 63.6)
Connections:
- J5 pad 1: /relay1/NC2 -> /relay1/NO2
- J5 pad 3: /relay1/NO2 -> /relay1/NC2
Routing:
- net /relay1/NO2: track 36.8 -> 44.1 mm
- net /relay1/NC2: track 37.4 -> 44.6 mm, vias 3 -> 4
Other:
- board size 56 x 17 mm -> 56 x 15 mm
- board text added: "COM"
- board text added: "NC"
- board text added: "NO"
- board text added: "OS-Relay General Purpose"
