File: hardware/General-Purpose-SMD/relay.kicad_sch (KiCad schematic)
At the start: 7 parts, among them J1 Screw_Terminal_01x03, J4 Screw_Terminal_01x03, J5 Screw_Terminal_01x03, K1 G6K-2F-Y-TR DC12, K2 G6K-2F-Y-TR DC12

Commit message: finalized relays repo. Yet to do manual. Release is ready togo
Connections:
- net NC2: now also J5.3 (Pin_3); no longer J5.1 (Pin_1)
- net NO2: now also J5.1 (Pin_1); no longer J5.3 (Pin_3)
Changed lines of the file:
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@@
 		(lib_id "Connector:Screw_Terminal_01x03")
 		(at 173.99 100.33 0)
+		(mirror x)
 		(unit 1)
 		(exclude_from_sim no)
@@
 		(on_board yes)
 		(dnp no)
-		(fields_autoplaced yes)
 		(property "Reference" "J5"
-			(at 176.53 100.3299 0)
+			(at 176.53 100.3301 0)
 			(effects
 				(font
@@
 		)
 		(property "Value" "Screw_Terminal_01x03"
-			(at 173.99 106.68 0)
+			(at 173.99 93.98 0)
 			(effects
 				(font
